Commit message: Updated Framework pick and place dry

File: urdf/fr_camera_gripper.urdf.xacro (robot description, xacro)
@@ -9,30 +9,39 @@
     <inertial>
       <origin
-        xyz="-1.5389E-05 0.0050006 0.035526"
-        rpy="0 0 0" />
-      <mass
-        value="0.60007" />
-      <inertia
-        ixx="0.00077666"
-        ixy="5.9011E-07"
-        ixz="4.3886E-07"
-        iyy="0.00066312"
-        iyz="-1.924E-05"
-        izz="0.00080686" />
-    </inertial>
-    <visual>
-      <origin
-        xyz="0 0 0"
-        rpy="0 0 0" />
-      <geometry>
-        <mesh
-          filename="package://fairino_description/meshes/fairino3_mt_v6/base_link.STL" />
-      </geometry>
-      <material
-        name="">
-        <color
-          rgba="1 1 1 1" />
-      </material>
-    </visual>
+        xyz="-0.00031896 -0.00029673 0.042463"
+        rpy="0 0 0" />
+      <mass
+        value="1.6185" />
+      <inertia
+        ixx="0.0030836"
+        ixy="1.5354E-05"
+        ixz="-1.9315E-05"
+        iyy="0.0030825"
+        iyz="-1.7918E-05"
+        izz="0.0045209" />
+    </inertial>
+    <visual>
+      <origin
+        xyz="0 0 0"
+        rpy="0 0 0" />
+      <geometry>
+        <mesh
+          filename="package://fairino_description/meshes/fairino5_v6/base_link.STL" />
+      </geometry>
+      <material
+        name="">
+        <color
+          rgba="0.89804 0.91765 0.92941 1" />
+      </material>
+    </visual>
+    <collision>
+      <origin
+        xyz="0 0 0"
+        rpy="0 0 0" />
+      <geometry>
+        <mesh
+          filename="package://fairino_description/meshes/fairino5_v6/base_link.STL" />
+      </geometry>
+    </collision>
   </link>
   <link
@@ -40,37 +49,46 @@
     <inertial>
       <origin
-        xyz="1.6205E-07 -0.0044494 0.00092552"
-        rpy="0 0 0" />
-      <mass
-        value="0.74148" />
-      <inertia
-        ixx="0.0011031"
-        ixy="2.2689E-08"
-        ixz="-5.9115E-09"
-        iyy="0.001042"
-        iyz="-3.0351E-06"
-        izz="0.00087179" />
-    </inertial>
-    <visual>
-      <origin
-        xyz="0 0 0"
-        rpy="0 0 0" />
-      <geometry>
-        <mesh
-          filename="package://fairino_description/meshes/fairino3_mt_v6/shoulder_link.STL" />
-      </geometry>
-      <material
-        name="">
-        <color
-          rgba="1 1 1 1" />
-      </material>
-    </visual>
+        xyz="5.0029E-07 -0.0040922 0.14629"
+        rpy="0 0 0" />
+      <mass
+        value="4.3771" />
+      <inertia
+        ixx="0.010731"
+        ixy="-8.0587E-09"
+        ixz="-3.6773E-08"
+        iyy="0.010408"
+        iyz="0.00012853"
+        izz="0.0081793" />
+    </inertial>
+    <visual>
+      <origin
+        xyz="0 0 0"
+        rpy="0 0 0" />
+      <geometry>
+        <mesh
+          filename="package://fairino_description/meshes/fairino5_v6/shoulder_link.STL" />
+      </geometry>
+      <material
+        name="">
+        <color
+          rgba="0.89804 0.91765 0.92941 1" />
+      </material>
+    </visual>
+    <collision>
+      <origin
+        xyz="0 0 0"
+        rpy="0 0 0" />
+      <geometry>
+        <mesh
+          filename="package://fairino_description/meshes/fairino5_v6/shoulder_link.STL" />
+      </geometry>
+    </collision>
   </link>
   <joint
-    name="joint1"
+    name="j1"
     type="revolute">
     <origin
-      xyz="0 0 0.1398"
-      rpy="-3.1416 0 3.1416" />
+      xyz="0 0 0"
+      rpy="0 0 0" />
     <parent
       link="base_link" />
@@ -78,10 +96,21 @@
       link="shoulder_link" />
     <axis
-      xyz="0 0 -1" />
+      xyz="0 0 1" />
     <limit
-      lower="-3.054"
-      upper="3.054"
-      effort="0"
-      velocity="2.618" />
+      lower="-3.0543"
+      upper="3.0543"
+      effort="150"
+      velocity="3.15" />
+    <calibration
+      rising="0"
+      falling="0" />
+    <dynamics
+      damping="0"
+      friction="0" />
+    <safety_controller
+      soft_lower_limit="-3.0543"
+      soft_upper_limit="3.0543"
+      k_position="15"
+      k_velocity="10" />
   </joint>
   <link
@@ -89,37 +118,46 @@
     <inertial>
       <origin
-        xyz="-0.140004201806272 5.58207727460597E-05 -0.00156100739557976"
-        rpy="0 0 0" />
-      <mass
-        value="2.23321682714675" />
-      <inertia
-        ixx="0.00277222130924851"
-        ixy="-1.37828945216777E-07"
-        ixz="3.33442608957987E-06"
-        iyy="0.0336038296729029"
-        iyz="2.35299017265147E-05"
-        izz="0.0329310083460027" />
-    </inertial>
-    <visual>
-      <origin
-        xyz="0 0 0"
-        rpy="0 0 0" />
-      <geometry>
-        <mesh
-          filename="package://fairino_description/meshes/fairino3_mt_v6/upperarm_link.STL" />
-      </geometry>
-      <material
-        name="">
-        <color
-          rgba="1 1 1 1" />
-      </material>
-    </visual>
+        xyz="-0.2125 -5.7643E-09 0.1346"
+        rpy="0 0 0" />
+      <mass
+        value="14.458" />
+      <inertia
+        ixx="0.028392"
+        ixy="-1.337E-07"
+        ixz="-3.9895E-09"
+        iyy="0.4559"
+        iyz="4.214E-08"
+        izz="0.44974" />
+    </inertial>
+    <visual>
+      <origin
+        xyz="0 0 0"
+        rpy="0 0 0" />
+      <geometry>
+        <mesh
+          filename="package://fairino_description/meshes/fairino5_v6/upperarm_link.STL" />
+      </geometry>
+      <material
+        name="">
+        <color
+          rgba="0.89804 0.91765 0.92941 1" />
+      </material>
+    </visual>
+    <collision>
+      <origin
+        xyz="0 0 0"
+        rpy="0 0 0" />
+      <geometry>
+        <mesh
+          filename="package://fairino_description/meshes/fairino5_v6/upperarm_link.STL" />
+      </geometry>
+    </collision>
   </link>
   <joint
-    name="joint2"
+    name="j2"
     type="revolute">
     <origin
-      xyz="-1.2826E-05 -0.114 0"
-      rpy="-1.6057 0 3.1416" />
+      xyz="0 0 0.152"
+      rpy="1.5708 0 0" />
     <parent
       link="shoulder_link" />
@@ -127,10 +165,21 @@
       link="upperarm_link" />
     <axis
-      xyz="0.00011251 -0.034899 0.99939" />
+      xyz="0 0 1" />
     <limit
       lower="-4.6251"
       upper="1.4835"
-      effort="0"
-      velocity="2.618" />
+      effort="150"
+      velocity="3.15" />
+    <calibration
+      rising="0"
+      falling="0" />
+    <dynamics
+      damping="0"
+      friction="0" />
+    <safety_controller
+      soft_lower_limit="-4.6251"
+      soft_upper_limit="1.4835"
+      k_position="15"
+      k_velocity="10" />
   </joint>
   <link
@@ -138,37 +187,46 @@
     <inertial>
       <origin
-        xyz="0.128489459057861 0.00376680150361507 0.10785794491905"
-        rpy="0 0 0" />
-      <mass
-        value="1.44662851848972" />
-      <inertia
-        ixx="0.00140089380811807"
-        ixy="-3.09715756532135E-05"
-        ixz="-0.000886845494769602"
-        iyy="0.015239432128819"
-        iyz="-1.00154489220657E-05"
-        izz="0.0149528743879964" />
-    </inertial>
-    <visual>
-      <origin
-        xyz="0 0 0"
-        rpy="0 0 0" />
-      <geometry>
-        <mesh
-          filename="package://fairino_description/meshes/fairino3_mt_v6/forearm_link.STL" />
-      </geometry>
-      <material
-        name="">
-        <color
-          rgba="1 1 1 1" />
-      </material>
-    </visual>
+        xyz="-0.18793 -8.4503E-07 0.0066357"
+        rpy="0 0 0" />
+      <mass
+        value="7.6737" />
+      <inertia
+        ixx="0.0085096"
+        ixy="2.1613E-06"
+        ixz="-0.0068678"
+        iyy="0.16971"
+        iyz="3.7086E-08"
+        izz="0.16854" />
+    </inertial>
+    <visual>
+      <origin
+        xyz="0 0 0"
+        rpy="0 0 0" />
+      <geometry>
+        <mesh
+          filename="package://fairino_description/meshes/fairino5_v6/forearm_link.STL" />
+      </geometry>
+      <material
+        name="">
+        <color
+          rgba="0.89804 0.91765 0.92941 1" />
+      </material>
+    </visual>
+    <collision>
+      <origin
+        xyz="0 0 0"
+        rpy="0 0 0" />
+      <geometry>
+        <mesh
+          filename="package://fairino_description/meshes/fairino5_v6/forearm_link.STL" />
+      </geometry>
+    </collision>
   </link>
   <joint
-    name="joint3"
+    name="j3"
     type="revolute">
     <origin
-      xyz="-0.28 0 3.1484E-05"
-      rpy="3.1416 0 3.1416" />
+      xyz="-0.425 0 0"
+      rpy="0 0 0" />
     <parent
       link="upperarm_link" />
@@ -176,10 +234,21 @@
       link="forearm_link" />
     <axis
-      xyz="0.00011251 0.034899 -0.99939" />
+      xyz="0 0 1" />
     <limit
-      lower="-2.618"
-      upper="2.618"
-      effort="0"
-      velocity="2.618" />
+      lower="-2.8274"
+      upper="2.8274"
+      effort="150"
+      velocity="3.15" />
+    <calibration
+      rising="0"
+      falling="0" />
+    <dynamics
+      damping="0"
+      friction="0" />
+    <safety_controller
+      soft_lower_limit="-2.8274"
+      soft_upper_limit="2.8274"
+      k_position="15"
+      k_velocity="10" />
   </joint>
   <link
@@ -187,36 +256,45 @@
     <inertial>
       <origin
-        xyz="-1.19852325169978E-05 -0.00486839591464538 -0.0978878853744289"
-        rpy="0 0 0" />
-      <mass
-        value="0.547616738862515" />
-      <inertia
-        ixx="0.000678878371004643"
-        ixy="-1.94106898510714E-10"
-        ixz="1.6479628472316E-08"
-        iyy="0.000507186880949965"
-        iyz="1.50098142579532E-06"
-        izz="0.000640889543804497" />
-    </inertial>
-    <visual>
-      <origin
-        xyz="0 0 0"
-        rpy="0 0 0" />
-      <geometry>
-        <mesh
-          filename="package://fairino_description/meshes/fairino3_mt_v6/wrist1_link.STL" />
-      </geometry>
-      <material
-        name="">
-        <color
-          rgba="1 1 1 1" />
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